File: Hardware/SmartSafeRev2/SmartSafeRev2.kicad_sch (KiCad schematic)
At the start: 16 parts

Commit message: Kicad Schematic updated
Parts:
- removed U?: DS1307_RTC_Module, symbol SmartSafeLibrary:DS1307_RTC_Module
Other:
- note removed: "I2C SCL"
- note removed: "I2C SDA"
- note removed: "RTC"
- note removed: "RTC Port"

Commit message: Schematic update
Parts:
- removed D?: Blue, symbol Device:LED
- removed R? (x4): 1k, symbol Device:R
- removed R?: 330, symbol Device:R
- added D1, D2, D3, D4: Blue, symbol Device:LED
- added R1, R2, R3, R4: 330, symbol Device:R
- added R5, R6, R7, R8: 1M, symbol Device:R
- R?: value 1k -> 1M
Connections:
- net +3V3: now also R5.1, R6.1, R7.1, R8.1
- net GND: now also D1.1 (K), D2.1 (K), D3.1 (K), D4.1 (K)
- net P4.0: now also R8.2
- net P4.1: now also R7.2
- net P4.2: now also R6.2
- net P4.3: now also R5.2
- new net: D1.2 (A), R1.2
- new net: D2.2 (A), R2.2
- new net: D4.2 (A), R4.2
- new net: D3.2 (A), R3.2
- new net P5.0: R2.1
- new net P5.1: R1.1
- new net P5.2: R4.1
- new net P5.4: R3.1
Other:
- note added: "Bluetooth Pins"
- note added: "Code Indicator LEDs"
- note added: "Keypad Pins"
- note added: "LED Pins"
- note added: "Open/Close Indicator LEDs"
- note added: "RTC Pin"
- note added: "Servo Pin"
- note added: "Switch Pin"
- note removed: "BlueTooth Port"
- note removed: "LED Port"
- note removed: "LEDs"
- note removed: "Microcontroller Pins"
- note removed: "Servo Port"
- note removed: "Switch Port"
- moved on the sheet: M?, R?, SW?, U?

Commit message: Final Commit
- Finishing Touches
Parts:
- added C1: 100nF, symbol Device:C
Connections:
- net GND: now also C1.2
- net P2.3: now also C1.1
- net P6.7 renamed P2.6
Other:
- note added: "RTC"
Changed lines of the file:
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@@
+    (stroke (width 0) (type default))
+  )
+  (wire (pts (xy 163.576 71.628) (xy 163.576 76.454))
     (stroke (width 0) (type default))
   )
@@
     (stroke (width 0) (type default))
   )
+  (wire (pts (xy 163.576 84.074) (xy 163.576 89.408))
+    (stroke (width 0) (type default))
+  )
   (wire (pts (xy 262.89 152.146) (xy 262.89 160.274))
     (stroke (width 0) (type default))
@@
     (fill (type none))
   )
+  (rectangle (start 151.638 65.786) (end 177.292 99.568)
+    (stroke (width 0) (type default))
+    (fill (type none))
+  )
   (rectangle (start 19.025 38.1) (end 48.025 75.1)
     (stroke (width 0) (type default))
@@
     (effects (font (size 1.27 1.27)) (justify left bottom))
   )
+  (text "RTC" (at 160.782 65.278 0)
+    (effects (font (size 1.27 1.27)) (justify left bottom))
+  )
   (text "UART Rx" (at 80.383 93.759 0)
     (effects (font (size 1.27 1.27)) (justify left bottom))
@@
     (effects (font (size 1.27 1.27)) (justify left bottom))
   )
-  (label "P6.7" (at 73.926 136.351 0) (fields_autoplaced)
+  (label "P2.6" (at 73.926 136.351 0) (fields_autoplaced)
     (effects (font (size 1.27 1.27)) (justify left bottom))
   )
@@
     (effects (font (size 1.27 1.27)) (justify left bottom))
   )
+  (label "P2.3" (at 163.576 71.628 0) (fields_autoplaced)
+    (effects (font (size 1.27 1.27)) (justify left bottom))
+  )
   (label "P5.4" (at 151.511 114.935 180) (fields_autoplaced)
     (effects (font (size 1.27 1.27)) (justify right bottom))
@@
     (effects (font (size 1.27 1.27)) (justify right bottom))
   )
-  (label "P6.7" (at 216.408 67.818 0) (fields_autoplaced)
+  (label "P2.6" (at 216.408 67.818 0) (fields_autoplaced)
     (effects (font (size 1.27 1.27)) (justify left bottom))
   )
@@
     )
   )
-  (global_label "P6.7" (shape input) (at 64.528 136.351 180) (fields_autoplaced)
-    (effects (font (size 1.27 1.27)) (justify right))
-    (property "Intersheetrefs" "${INTERSHEET_REFS}" (at 57.8211 136.2716 0)
+  (global_label "P2.6" (shape input) (at 64.528 136.351 180) (fields_autoplaced)
+    (effects (font (size 1.27 1.27)) (justify right))
+    (property "Intersheetrefs" "${INTERSHEET_REFS}" (at 57.249 136.351 0)
       (effects (font (size 1.27 1.27)) (justify right) hide)
     )
@@
         (path "/e1f8f346-d680-4c02-a353-e2351bb45f33"
           (reference "R6") (unit 1)
+        )
+      )
+    )
+  )
+  (symbol (lib_id "Device:C") (at 163.576 80.264 0) (unit 1)
+    (in_bom yes) (on_board yes) (dnp no) (fields_autoplaced)
+    (property "Reference" "C1" (at 167.64 78.994 0)
+      (effects (font (size 1.27 1.27)) (justify left))
+    )
+    (property "Value" "100nF" (at 167.64 81.534 0)
+      (effects (font (size 1.27 1.27)) (justify left))
+    )
+    (property "Footprint" "" (at 164.5412 84.074 0)
+      (effects (font (size 1.27 1.27)) hide)
+    )
+    (property "Datasheet" "~" (at 163.576 80.264 0)
+      (effects (font (size 1.27 1.27)) hide)
+    )
+    (pin "1")
+    (pin "2")
+    (instances
+      (project "SmartSafeRev2"
+        (path "/e1f8f346-d680-4c02-a353-e2351bb45f33"
+          (reference "C1") (unit 1)
         )
       )
@@
         )
       )
+    )
+  )
+  (symbol (lib_id "power:GND") (at 163.576 89.408 0) (unit 1)
+    (in_bom yes) (on_board yes) (dnp no) (fields_autoplaced)
+    (property "Reference" "#PWR09" (at 163.576 95.758 0)
+      (effects (font (size 1.27 1.27)) hide)
+    )
+    (property "Value" "GND" (at 163.576 94.488 0)
+      (effects (font (size 1.27 1.27)))
+    )
+    (property "Footprint" "" (at 163.576 89.408 0)
+      (effects (font (size 1.27 1.27)) hide)
+    )
+    (property "Datasheet" "" (at 163.576 89.408 0)
+      (effects (font (size 1.27 1.27)) hide)
+    )
+    (pin "1")
+    (instances
+      (project "SmartSafeRev2"
+        (path "/e1f8f346-d680-4c02-a353-e2351bb45f33"
+          (reference "#PWR09") (unit 1)
+        )
+      )
